File: ahrs-can-adapter.kicad_pcb (KiCad board)
At the start: 2 copper layers, 61.3 x 77 mm, 48 parts, among them J1 Flight Power, J2 Flight Telem, J3 CAN IN, J4 CAN OUT, SW1 Reset, U1 MPM3610-adafruit 5V, U2 UA78M33CDCYR, U3 LTC2875-S8, U4 STM32G474RET6, U5 VCAN26A2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

Commit message: Changed telemetry uart pins
Connections:
- U4 pad 14: TX -> unconnected-(U4-PA2-Pad14)
- U4 pad 17: RX -> unconnected-(U4-PA3-Pad17)
- U4 pad 52: unconnected-(U4-PC10-Pad52) -> TX
- U4 pad 53: unconnected-(U4-PC11-Pad53) -> RX
Routing:
- net TX: track 22.4 -> 42.4 mm, vias 0 -> 2
- net RX: track 13.4 -> 28.0 mm
- net Current: track 53.6 -> 52.6 mm
